Commit message: Reset Postion need to fix

File: aragog_urdf/urdf/aragog.urdf (robot description, URDF)
Before this commit: robot mercury_urdf, 15 links, 14 joints
Links:
- link BLA: geometry collision mesh filename=package://aragog_urdf/meshes/BLA.STL; visual mesh filename=package://aragog_urdf/meshes/BLA.STL
- link BLH: geometry collision mesh filename=package://aragog_urdf/meshes/BLH.STL; visual mesh filename=package://aragog_urdf/meshes/BLH.STL
- link BLK: geometry collision mesh filename=package://aragog_urdf/meshes/BLK.STL; visual mesh filename=package://aragog_urdf/meshes/BLK.STL
- link BRA: geometry collision mesh filename=package://aragog_urdf/meshes/BRA.STL; visual mesh filename=package://aragog_urdf/meshes/BRA.STL
- link BRH: geometry collision mesh filename=package://aragog_urdf/meshes/BRH.STL; visual mesh filename=package://aragog_urdf/meshes/BRH.STL
- link BRK: geometry collision mesh filename=package://aragog_urdf/meshes/BRK.STL; visual mesh filename=package://aragog_urdf/meshes/BRK.STL
- link Back_module: geometry collision mesh filename=package://aragog_urdf/meshes/Back_module.STL; visual mesh filename=package://aragog_urdf/meshes/Back_module.STL
- link FLA: geometry collision mesh filename=package://aragog_urdf/meshes/FLA.STL; visual mesh filename=package://aragog_urdf/meshes/FLA.STL
- link FLH: geometry collision mesh filename=package://aragog_urdf/meshes/FLH.STL; visual mesh filename=package://aragog_urdf/meshes/FLH.STL
- link FLK: geometry collision mesh filename=package://aragog_urdf/meshes/FLK.STL; visual mesh filename=package://aragog_urdf/meshes/FLK.STL
- link FRA: geometry collision mesh filename=package://aragog_urdf/meshes/FRA.STL; visual mesh filename=package://aragog_urdf/meshes/FRA.STL
- link FRH: geometry collision mesh filename=package://aragog_urdf/meshes/FRH.STL; visual mesh filename=package://aragog_urdf/meshes/FRH.STL
- link FRK: geometry collision mesh filename=package://aragog_urdf/meshes/FRK.STL; visual mesh filename=package://aragog_urdf/meshes/FRK.STL
- link Front_module: geometry collision mesh filename=package://aragog_urdf/meshes/Front_module.STL; visual mesh filename=package://aragog_urdf/meshes/Front_module.STL
- link base_link: geometry collision mesh filename=package://aragog_urdf/meshes/base_link.STL; visual mesh filename=package://aragog_urdf/meshes/base_link.STL

Commit message: Added different morphologies and reset morphology function

File: aragog_urdf/urdf/aragog.urdf (robot description, URDF)
Before this commit: robot aragog_urdf, 15 links, 14 joints
Joints:
- joint BLH_joint: axis 0 0 -1 -> 0 0 1
- joint BRH_joint: axis 0 0 -1 -> 0 0 1
- joint FLH_joint: axis 0 0 -1 -> 0 0 1
- joint FRH_joint: axis 0 0 -1 -> 0 0 1
